File: vfd/untitled.sch (EAGLE design)
At the start: 80 parts, among them IC1 FSBB30CH60, IC2 74HCT04D, T1 BC547, X3 5202-06-N-02

Commit message: update trafo
trafo 15v
Parts:
- added B2: (no value), rectifier:S41
- added C32, C33, C34: (no value), rcl:CPOL-EUB45181A
- added IC3: 15, v-reg:78MXXL
- added IC4: 5, v-reg:78MXXL
- added TR1: (no value), trafo:EI30-1
Connections:
- new net N$1: B2.AC1, TR1.S4
- new net N$11: B2.-, C32.-, C33.-, C34.-, IC3.GND, IC4.GND
- new net N$3: B2.AC2, TR1.S3
- new net N$7: B2.+, C34.+, IC3.IN
- net +15V: now also C32.+, IC3.OUT, IC4.IN
- net +5V: now also C33.+, IC4.OUT
- net L: now also TR1.P1
- net N: now also TR1.P2
Changed lines of the file:
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@@
 <part name="FRAME1" library="frames" library_urn="urn:adsk.eagle:library:229" deviceset="A3L-LOC" device=""/>
 <part name="X3" library="con-ebyelectro" library_urn="urn:adsk.eagle:library:141" deviceset="5202-06-N-02" device="" package3d_urn="urn:adsk.eagle:package:6687/1"/>
+<part name="TR1" library="trafo" library_urn="urn:adsk.eagle:library:394" deviceset="EI30-1" device="" package3d_urn="urn:adsk.eagle:package:28333/1"/>
+<part name="B2" library="rectifier" library_urn="urn:adsk.eagle:library:336" deviceset="S41" device="" package3d_urn="urn:adsk.eagle:package:23883/1"/>
+<part name="IC3" library="v-reg" library_urn="urn:adsk.eagle:library:409" deviceset="78MXXL" device="" package3d_urn="urn:adsk.eagle:package:30356/1" value="15"/>
+<part name="IC4" library="v-reg" library_urn="urn:adsk.eagle:library:409" deviceset="78MXXL" device="" package3d_urn="urn:adsk.eagle:package:30356/1" value="5"/>
+<part name="C32" library="rcl" library_urn="urn:adsk.eagle:library:334" deviceset="CPOL-EU" device="B45181A" package3d_urn="urn:adsk.eagle:package:23316/1"/>
+<part name="C33" library="rcl" library_urn="urn:adsk.eagle:library:334" deviceset="CPOL-EU" device="B45181A" package3d_urn="urn:adsk.eagle:package:23316/1"/>
+<part name="C34" library="rcl" library_urn="urn:adsk.eagle:library:334" deviceset="CPOL-EU" device="B45181A" package3d_urn="urn:adsk.eagle:package:23316/1"/>
 </parts>
 <sheets>
@@
 <attribute name="NAME" x="67.691" y="138.811" size="1.778" layer="95" rot="MR0"/>
 </instance>
+<instance part="TR1" gate="1" x="78.74" y="152.4" smashed="yes">
+<attribute name="NAME" x="76.2" y="159.766" size="1.778" layer="95"/>
+<attribute name="VALUE" x="76.2" y="141.605" size="1.778" layer="96"/>
+</instance>
+<instance part="B2" gate="1" x="-2.54" y="157.48" smashed="yes">
+<attribute name="NAME" x="0" y="160.02" size="1.778" layer="95"/>
+<attribute name="VALUE" x="0" y="153.67" size="1.778" layer="96"/>
+</instance>
+<instance part="IC3" gate="A" x="15.24" y="157.48" smashed="yes">
+<attribute name="NAME" x="17.78" y="149.86" size="1.778" layer="95"/>
+<attribute name="VALUE" x="17.78" y="147.32" size="1.778" layer="96"/>
+</instance>
+<instance part="IC4" gate="A" x="35.56" y="157.48" smashed="yes">
+<attribute name="NAME" x="38.1" y="149.86" size="1.778" layer="95"/>
+<attribute name="VALUE" x="38.1" y="147.32" size="1.778" layer="96"/>
+</instance>
+<instance part="C32" gate="G$1" x="25.4" y="154.94" smashed="yes">
+<attribute name="NAME" x="26.543" y="155.4226" size="1.778" layer="95"/>
+<attribute name="VALUE" x="26.543" y="150.3426" size="1.778" layer="96"/>
+</instance>
+<instance part="C33" gate="G$1" x="45.72" y="154.94" smashed="yes">
+<attribute name="NAME" x="46.863" y="155.4226" size="1.778" layer="95"/>
+<attribute name="VALUE" x="46.863" y="150.3426" size="1.778" layer="96"/>
+</instance>
+<instance part="C34" gate="G$1" x="5.08" y="154.94" smashed="yes">
+<attribute name="NAME" x="6.223" y="155.4226" size="1.778" layer="95"/>
+<attribute name="VALUE" x="6.223" y="150.3426" size="1.778" layer="96"/>
+</instance>
 </instances>
 <busses>
@@
 <wire x1="48.26" y1="86.36" x2="50.8" y2="86.36" width="0.1524" layer="91"/>
 <junction x="50.8" y="86.36"/>
+</segment>
+<segment>
+<pinref part="IC3" gate="A" pin="OUT"/>
+<pinref part="C32" gate="G$1" pin="+"/>
+<wire x1="22.86" y1="157.48" x2="25.4" y2="157.48" width="0.1524" layer="91"/>
+<pinref part="IC4" gate="A" pin="IN"/>
+<wire x1="25.4" y1="157.48" x2="27.94" y2="157.48" width="0.1524" layer="91"/>
+<junction x="25.4" y="157.48"/>
+<label x="22.86" y="160.02" size="1.778" layer="95"/>
 </segment>
 </net>
@@
 <pinref part="OK5" gate="A" pin="A1"/>
 </segment>
+<segment>
+<pinref part="IC4" gate="A" pin="OUT"/>
+<pinref part="C33" gate="G$1" pin="+"/>
+<wire x1="43.18" y1="157.48" x2="45.72" y2="157.48" width="0.1524" layer="91"/>
+<label x="43.18" y="160.02" size="1.778" layer="95"/>
+</segment>
 </net>
 <net name="N$27" class="0">
@@
 <label x="78.74" y="147.32" size="1.778" layer="95"/>
 <pinref part="X3" gate="-5" pin="1"/>
+<pinref part="TR1" gate="1" pin="P2"/>
+<junction x="73.66" y="144.78"/>
 </segment>
 </net>
@@
 <pinref part="F2" gate="1" pin="1"/>
 <pinref part="X3" gate="-4" pin="1"/>
+<pinref part="TR1" gate="1" pin="P1"/>
+<junction x="73.66" y="157.48"/>
 </segment>
 </net>
@@
 </segment>
 </net>
+<net name="N$1" class="0">
+<segment>
+<pinref part="TR1" gate="1" pin="S4"/>
+<pinref part="B2" gate="1" pin="AC1"/>
+<wire x1="86.36" y1="154.94" x2="86.36" y2="162.56" width="0.1524" layer="91"/>
+<wire x1="86.36" y1="162.56" x2="-2.54" y2="162.56" width="0.1524" layer="91"/>
+</segment>
+</net>
+<net name="N$3" class="0">
+<segment>
+<pinref part="TR1" gate="1" pin="S3"/>
+<wire x1="86.36" y1="147.32" x2="86.36" y2="129.54" width="0.1524" layer="91"/>
+<pinref part="B2" gate="1" pin="AC2"/>
+<wire x1="86.36" y1="129.54" x2="-2.54" y2="129.54" width="0.1524" layer="91"/>
+<wire x1="-2.54" y1="129.54" x2="-2.54" y2="152.4" width="0.1524" layer="91"/>
+</segment>
+</net>
+<net name="N$7" class="0">
+<segment>
+<pinref part="IC3" gate="A" pin="IN"/>
+<pinref part="C34" gate="G$1" pin="+"/>
+<wire x1="7.62" y1="157.48" x2="5.08" y2="157.48" width="0.1524" layer="91"/>
+<pinref part="B2" gate="1" pin="+"/>
+<wire x1="2.54" y1="157.48" x2="5.08" y2="157.48" width="0.1524" layer="91"/>
+<junction x="5.08" y="157.48"/>
+</segment>
+</net>
+<net name="N$11" class="0">
+<segment>
+<pinref part="C33" gate="G$1" pin="-"/>
+<pinref part="IC4" gate="A" pin="GND"/>
+<wire x1="45.72" y1="149.86" x2="35.56" y2="149.86" width="0.1524" layer="91"/>
+<pinref part="C32" gate="G$1" pin="-"/>
+<wire x1="35.56" y1="149.86" x2="25.4" y2="149.86" width="0.1524" layer="91"/>
+<junction x="35.56" y="149.86"/>
+<pinref part="C34" gate="G$1" pin="-"/>
+<wire x1="25.4" y1="149.86" x2="15.24" y2="149.86" width="0.1524" layer="91"/>
+<junction x="25.4" y="149.86"/>
+<pinref part="IC3" gate="A" pin="GND"/>
+<wire x1="15.24" y1="149.86" x2="5.08" y2="149.86" width="0.1524" layer="91"/>
+<junction x="15.24" y="149.86"/>
+<pinref part="B2" gate="1" pin="-"/>
+<wire x1="-7.62" y1="157.48" x2="-7.62" y2="149.86" width="0.1524" layer="91"/>
+<wire x1="-7.62" y1="149.86" x2="5.08" y2="149.86" width="0.1524" layer="91"/>
+<junction x="5.08" y="149.86"/>
+</segment>
+</net>
 </nets>
 </sheet>
+<sheet>
+<plain>
+</plain>
+<instances>
+</instances>
+<busses>
+</busses>
+<nets>
+</nets>
+</sheet>
